File: sun3_60.kicad_pcb (KiCad board)
At the start: 4 copper layers, 229 parts, among them J1 KB/Mouse, J11 Conn_01x04_Pin, J2 Serial A/B, J200 SW_Push_SPDT, J3 Conn_01x09_Pin, K199 10UF, K500 10 uF, K900 1000uF, K901 1000uF, K903 1000uF, K904 1000uF, U100 68020, U102 PAL16L8, U103 PAL16L8, U104 74F04, U106 PAL16L8, U107 PAL20X10, U108 74F00, U110 40.000 Mhz, U113 74AS74, U114 74F175, U115 74LS590, U122 ALS374, U123 ALS373, U130 74F374, U131 PAL16R6, U132 ALS244, U199 7705, U200 7188, U2003 74AS04, U2004 74LS125, U201 7188, U202 2168, U203 2168, U205 2168, U206 2168, U207 2168, U208 2168, U210 LS2518, U212 ALS245, U213 ALS245, U215 ALS245, U217 ALS245, U218 ALS245, U223 74F534, U224 AM27S19, U225 ALS273, U226 ALS373, U227 ALS273, U228 LED_Block, U229 LED_Block, U230 PAL16L8, U231 PAL16L8, U232 PAL16L8, U300 27512, U301 28C16, U302 7170, U303 32768Hz, U304 ALS273, U305 ALS373, U307 PAL20L8, U309 3-VOLT, U310 PAL20L8, U311 PAL20L8, U312 PAL8L14, U313 PAL16R4, U400 Z8530, U401 Z8530, U402 4.9152 Mhz, U404 74LS04, U408 74LS04, U500 AM7990, U501 AM7992, U502 20 Mhz, U503 TRANSF, U510 ALS373, U511 ALS373, U512 ALS373, U514 ALS652, U515 ALS652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

Commit message: Initial layout
- Lay out the PCB to match the original board sans the missing components. No routing yet.
- Pick standard library footprints instead of custom ones for some components.
- Change some ERC errors into warnings - like output pin connected to output pin.
- Change resistor network S200 from DIP to SIP type.
- Set Serial keyboard/mouse section to “Do Not Populate” to gain some space, and it wasn’t going to be used with no video possible anyway. However, in knockout testing with 3.0.1 boot PROM self tests pass, then a warning message tests were interrupted is emitted. Tests then re-run, but system hangs before giving a prompt.
- Fix the LED blocks for the diag register to match the original Dialight 555-4003 part.
Parts:
- removed J1: KB/Mouse, Connector_PinHeader_2.54mm:PinHeader_1x05_P2.54mm_Vertical
- removed S401: 4.7K Ohm, Resistor_THT:R_Array_SIP8
- removed U400: Z8530, Package_DIP:DIP-40_W15.24mm
- removed U404: 74LS04, Package_DIP:DIP-14_W7.62mm
- J200: value SW_Push_SPDT -> DIAG
- J3: value Conn_01x09_Pin -> Ethernet
- S200: value R_Pack04 -> 68 Ohm; footprint sun3_60:DIP-8_296_ELL -> Resistor_THT:R_Array_SIP8
- U122, U123, U226, U305, U510, U511, U512, U720, U721, U722, U723: footprint sun3_60:ALS373 -> Package_DIP:DIP-20_W7.62mm
- U200, U201: footprint sun3_60:7188 -> Package_DIP:DIP-22_W7.62mm
- U202, U203, U205, U206, U207, U208: footprint sun3_60:2168 -> Package_DIP:DIP-20_W7.62mm
- U210: footprint sun3_60:LS2518 -> Package_DIP:DIP-16_W7.62mm
- U212, U213, U215, U217, U218: footprint sun3_60:ALS245 -> Package_DIP:DIP-20_W7.62mm
- U224: footprint sun3_60:AM27S19 -> Package_DIP:DIP-16_W7.62mm
- U225, U227, U304: footprint sun3_60:ALS273 -> Package_DIP:DIP-20_W7.62mm
- U228, U229: footprint Connector_PinHeader_1.00mm:PinHeader_2x04_P1.00mm_Vertical -> Connector_PinHeader_2.54mm:PinHeader_2x04_P2.54mm_Vertical
- moved U501 306.0 mm to (109.2, 337.8), turned to 90 degrees
- moved R502 296.1 mm to (180.3, 357.1), turned to 180 degrees
- moved U500 283.0 mm to (91.4, 313.4), turned to 90 degrees
- moved C502 279.4 mm to (162.6, 357.1)
- moved K903 275.0 mm to (213.4, 340.4)
- moved C503 274.4 mm to (157.5, 357.1), turned to 180 degrees
- moved R501 274.0 mm to (139.7, 343.2), turned to -90 degrees
- moved J3 272.8 mm to (104.1, 357.1), turned to 90 degrees
- moved C504 267.9 mm to (147.2, 357.1), turned to 180 degrees
- moved C500 263.6 mm to (152.4, 336.8)
- moved C505 261.7 mm to (137.2, 357.1), turned to 180 degrees
- moved C501 257.2 mm to (142.3, 336.8)
- moved J200 256.1 mm to (108.0, 344.2)
- moved S502 254.8 mm to (129.5, 322.6)
- moved U229 254.6 mm to (223.5, 355.6), turned to 90 degrees
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Connections:
- S200 pad 2: /sun3_60_mmu_diag/TYPE0X -> /sun3_60_eeprom/TYPE1
- S200 pad 3: /sun3_60_mmu_diag/ACCESSX -> /sun3_60_mmu_diag/TYPE0X
- S200 pad 4: /sun3_60_mmu_diag/MODIFYX -> /sun3_60_eeprom/TYPE0
- S200 pad 5: /sun3_60_mmu_diag/MODIFY -> /sun3_60_mmu_diag/ACCESSX
- S200 pad 7: /sun3_60_eeprom/TYPE0 -> /sun3_60_mmu_diag/MODIFYX
- S200 pad 8: /sun3_60_eeprom/TYPE1 -> /sun3_60_mmu_diag/MODIFY
- U228 pad 1: /sun3_60_mmu_diag/LED0 -> VCC
- U228 pad 2: VCC -> /sun3_60_mmu_diag/LED0
- U228 pad 3: /sun3_60_mmu_diag/LED1 -> VCC
- U228 pad 4: VCC -> /sun3_60_mmu_diag/LED1
- U228 pad 5: /sun3_60_mmu_diag/LED2 -> VCC
- U228 pad 6: VCC -> /sun3_60_mmu_diag/LED2
- U228 pad 7: /sun3_60_mmu_diag/LED3 -> VCC
- U228 pad 8: VCC -> /sun3_60_mmu_diag/LED3
- U229 pad 1: /sun3_60_mmu_diag/LED4 -> VCC
- U229 pad 2: VCC -> /sun3_60_mmu_diag/LED4
- U229 pad 3: /sun3_60_mmu_diag/LED5 -> VCC
- U229 pad 4: VCC -> /sun3_60_mmu_diag/LED5
- U229 pad 5: /sun3_60_mmu_diag/LED6 -> VCC
- U229 pad 6: VCC -> /sun3_60_mmu_diag/LED6
- U229 pad 7: /sun3_60_mmu_diag/LED7 -> VCC
- U229 pad 8: VCC -> /sun3_60_mmu_diag/LED7
