File: sun3_60_ethernet.kicad_sch (KiCad schematic)
At the start: 28 parts, among them J3 Conn_01x09_Pin, K500 10 uF, U500 AM7990, U501 AM7992, U502 20 Mhz, U503 TRANSF, U508 DG303A, U509 DG303A, U510 ALS373, U511 ALS373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

Commit message: Initial layout
- Lay out the PCB to match the original board sans the missing components. No routing yet.
- Pick standard library footprints instead of custom ones for some components.
- Change some ERC errors into warnings - like output pin connected to output pin.
- Change resistor network S200 from DIP to SIP type.
- Set Serial keyboard/mouse section to “Do Not Populate” to gain some space, and it wasn’t going to be used with no video possible anyway. However, in knockout testing with 3.0.1 boot PROM self tests pass, then a warning message tests were interrupted is emitted. Tests then re-run, but system hangs before giving a prompt.
- Fix the LED blocks for the diag register to match the original Dialight 555-4003 part.
Parts:
- J3: value Conn_01x09_Pin -> Ethernet
Changed lines of the file:
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@@
 		(fields_autoplaced yes)
 		(property "Reference" "J3"
-			(at 225.425 149.86 0)
+			(at 227.33 163.8299 0)
 			(effects
 				(font
 					(size 1.27 1.27)
 				)
+				(justify right)
 			)
 		)
-		(property "Value" "Conn_01x09_Pin"
-			(at 225.425 152.4 0)
+		(property "Value" "Ethernet"
+			(at 227.33 166.3699 0)
 			(effects
 				(font
 					(size 1.27 1.27)
 				)
+				(justify right)
 			)
 		)

Commit message: Routing
- Initial routing with standard 4 layers setup
- Add SIM holes
- Copper to edge clearance 1.0mm
- Relaxed the layout a little so the autorouter can have results
- Moved K500 to the ethernet section it belongs to, and changed type. Same for K199
Parts:
- K500: footprint Capacitor_THT:CP_Radial_D10.0mm_P5.00mm -> Capacitor_THT:CP_Radial_Tantal_D6.0mm_P2.50mm
Changed lines of the file:
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@@
 			)
 		)
-		(property "Footprint" "Capacitor_THT:CP_Radial_D10.0mm_P5.00mm"
+		(property "Footprint" "Capacitor_THT:CP_Radial_Tantal_D6.0mm_P2.50mm"
 			(at 87.63 208.28 0)
 			(effects
@@
 			)
 		)
-		(property "Datasheet" "~"
+		(property "Datasheet" "https://www.digikey.com/en/products/detail/kyocera-avx/TAP106M035SCS/1471228"
 			(at 87.63 208.28 0)
 			(effects
@@
 			(at 87.63 208.28 0)
 			(effects
+				(font
+					(size 1.27 1.27)
+				)
+				(hide yes)
+			)
+		)
+		(property "Field5" ""
+			(at 87.63 208.28 0)
+			(effects

Commit message: Clean up before reorganizing the folders. The schematics and PCB reflect the fixes discovered during the prototype build.
Parts:
- S502: value 1K Ohm -> 1k Ohm
Changed lines of the file:
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@@
 		(fields_autoplaced yes)
 		(property "Reference" "S502"
-			(at 340.6139 29.21 0)
+			(at 341.884 25.4 90)
 			(effects
 				(font
 					(size 1.27 1.27)
 				)
-				(justify right)
 			)
 		)
-		(property "Value" "1K Ohm"
-			(at 343.1539 29.21 0)
+		(property "Value" "1k Ohm"
+			(at 341.884 27.94 90)
 			(effects
 				(font
 					(size 1.27 1.27)
 				)
-				(justify right)
 			)
 		)
