File: sun3_60_memory.kicad_sch (KiCad schematic)
At the start: 10 parts, among them U104 74F04, U108 74F00, U600 74F04, U800 PAL16L8, U801 74AS257, U802 PAL20L8, U803 74F64, U804 74F64, U805 PAL16L8

Commit message: Clean up before reorganizing the folders. The schematics and PCB reflect the fixes discovered during the prototype build.
Other:
- note removed: "TODO: Check VCC"
Changed lines of the file:
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@@
-		)
-	)
-	(text "TODO: Check VCC"
-		(exclude_from_sim no)
-		(at 203.962 76.454 0)
-		(effects
-			(font
-				(size 1.27 1.27)
-			)
 		)
 	)
