File: sun3_60_serial.kicad_sch (KiCad schematic)
At the start: 9 parts, among them J1 KB/Mouse, J2 Serial A/B, U400 Z8530, U401 Z8530, U402 4.9152 Mhz, U404 74LS04, U408 74LS04

Commit message: Clean up before reorganizing the folders. The schematics and PCB reflect the fixes discovered during the prototype build.
Parts:
- removed U402: 4.9152 Mhz, Oscillator:Oscillator_DIP-8, symbol Oscillator:CXO_DIP8
- added U402: 4.9152 Mhz, Oscillator:Oscillator_DIP-14, symbol Oscillator:CXO_DIP14
- U404, U408: value 74LS04 -> 74ALS04
Connections:
- net GND: now also U402.7 (GND)
- net VCC: now also U402.14 (Vcc)
- net at U400.20 (PCLK), U401.20 (PCLK): now also U402.8 (OUT)
Changed lines of the file:
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@@
 			)
 		)
-		(property "Value" "74LS04"
+		(property "Value" "74ALS04"
 			(at 26.67 179.07 0)
 			(effects
@@
 	)
 	(symbol
+		(lib_id "Oscillator:CXO_DIP14")
+		(at 29.21 102.87 0)
+		(unit 1)
+		(exclude_from_sim no)
+		(in_bom yes)
+		(on_board yes)
+		(dnp no)
+		(fields_autoplaced yes)
+		(property "Reference" "U402"
+			(at 40.64 96.5514 0)
+			(effects
+				(font
+					(size 1.27 1.27)
+				)
+			)
+		)
+		(property "Value" "4.9152 Mhz"
+			(at 40.64 99.0914 0)
+			(effects
+				(font
+					(size 1.27 1.27)
+				)
+			)
+		)
+		(property "Footprint" "Oscillator:Oscillator_DIP-14"
+			(at 40.64 111.76 0)
+			(effects
+				(font
+					(size 1.27 1.27)
+				)
+				(hide yes)
+			)
+		)
+		(property "Datasheet" "http://cdn-reichelt.de/documents/datenblatt/B400/OSZI.pdf"
+			(at 26.67 102.87 0)
+			(effects
+				(font
+					(size 1.27 1.27)
+				)
+				(hide yes)
+			)
+		)
+		(property "Description" "Crystal Clock Oscillator, DIP14-style metal package"
+			(at 29.21 102.87 0)
+			(effects
+				(font
+					(size 1.27 1.27)
+				)
+				(hide yes)
+			)
+		)
+		(pin "14"
+		)
+		(pin "7"
+		)
+		(pin "1"
+		)
+		(pin "8"
+		)
+		(instances
+			(project ""
+				(path "/d6b5cf90-8df0-4384-868a-524abed7c432/054c9f34-4c69-4214-aead-9eddc8182f56"
+					(reference "U402")
+					(unit 1)
+				)
+			)
+		)
+	)
+	(symbol
 		(lib_id "74xx:74LS04")
 		(at 269.24 139.7 0)
@@
 			)
 		)
-		(property "Value" "74LS04"
+		(property "Value" "74ALS04"
 			(at 269.24 133.35 0)
 			(effects
@@
 					(reference "U408")
 					(unit 5)
-				)
-			)
-		)
-	)
-	(symbol
-		(lib_id "Oscillator:CXO_DIP8")
-		(at 29.21 102.87 0)
-		(unit 1)
-		(exclude_from_sim no)
-		(in_bom yes)
-		(on_board yes)
-		(dnp no)
-		(fields_autoplaced yes)
-		(property "Reference" "U402"
-			(at 41.91 96.5514 0)
-			(effects
-				(font
-					(size 1.27 1.27)
-				)
-			)
-		)
-		(property "Value" "4.9152 Mhz"
-			(at 41.91 99.0914 0)
-			(effects
-				(font
-					(size 1.27 1.27)
-				)
-			)
-		)
-		(property "Footprint" "Oscillator:Oscillator_DIP-8"
-			(at 40.64 111.76 0)
-			(effects
-				(font
-					(size 1.27 1.27)
-				)
-				(hide yes)
-			)
-		)
-		(property "Datasheet" "http://cdn-reichelt.de/documents/datenblatt/B400/OSZI.pdf"
-			(at 26.67 102.87 0)
-			(effects
-				(font
-					(size 1.27 1.27)
-				)
-				(hide yes)
-			)
-		)
-		(property "Description" "Crystal Clock Oscillator, DIP8-style metal package"
-			(at 29.21 102.87 0)
-			(effects
-				(font
-					(size 1.27 1.27)
-				)
-				(hide yes)
-			)
-		)
-		(pin "8"
-		)
-		(pin "4"
-		)
-		(pin "1"
-		)
-		(pin "5"
-		)
-		(instances
-			(project ""
-				(path "/d6b5cf90-8df0-4384-868a-524abed7c432/054c9f34-4c69-4214-aead-9eddc8182f56"
-					(reference "U402")
-					(unit 1)
 				)
 			)
@@
 			)
 		)
-		(property "Value" "74LS04"
+		(property "Value" "74ALS04"
 			(at 121.92 163.83 0)
 			(effects
@@
 			)
 		)
-		(property "Value" "74LS04"
+		(property "Value" "74ALS04"
 			(at 270.51 33.0199 0)
 			(effects
@@
 			)
 		)
-		(property "Value" "74LS04"
+		(property "Value" "74ALS04"
 			(at 233.68 99.06 0)
 			(effects
@@
 			)
 		)
-		(property "Value" "74LS04"
+		(property "Value" "74ALS04"
 			(at 80.01 146.05 0)
 			(effects
@@
 			)
 		)
-		(property "Value" "74LS04"
+		(property "Value" "74ALS04"
 			(at 80.01 130.81 0)
 			(effects
@@
 		(on_board yes)
 		(dnp no)
-		(fields_autoplaced yes)
 		(property "Reference" "U408"
 			(at 214.63 58.42 0)
@@
 			)
 		)
-		(property "Value" "74LS04"
+		(property "Value" "74ALS04"
 			(at 214.63 60.96 0)
 			(effects
@@
 		(on_board yes)
 		(dnp no)
-		(fields_autoplaced yes)
 		(property "Reference" "U408"
 			(at 214.63 33.02 0)
@@
 			)
 		)
-		(property "Value" "74LS04"
+		(property "Value" "74ALS04"
 			(at 214.63 35.56 0)
 			(effects
@@
 			)
 		)
-		(property "Value" "74LS04"
+		(property "Value" "74ALS04"
 			(at 29.21 143.5099 0)
 			(effects
@@
 			)
 		)
-		(property "Value" "74LS04"
+		(property "Value" "74ALS04"
 			(at 48.26 179.07 0)
 			(effects
@@
 			)
 		)
-		(property "Value" "74LS04"
+		(property "Value" "74ALS04"
 			(at 233.68 76.2 0)
 			(effects
@@
 			)
 		)
-		(property "Value" "74LS04"
+		(property "Value" "74ALS04"
 			(at 269.24 148.59 0)
 			(effects
@@
 			)
 		)
-		(property "Value" "74LS04"
+		(property "Value" "74ALS04"
 			(at 121.92 147.32 0)
 			(effects
